File: 555-temporizador-r01.kicad_pcb (KiCad board)
At the start: 2 copper layers, 49.5 x 49.3 mm, 12 parts, among them J1 Saída Piscante, J2 Alimentação, J3 Disparo, SW1 SW_Push, U1 NE555

Commit message: generated gerbers r02
Other:
- net class Default removed
